Commit message: Add Nav2 + SLAM configs, custom room world, motor/URDF fixes

File: src/my_turtlebot_pkg/urdf/turtlebot.urdf.xacro (robot description, xacro)
@@ -156,5 +156,5 @@
   <link name="${prefix}_motor_link">
     <visual>
-      <origin xyz="0.0155 ${reflect * -0.018} 0" rpy="0 ${PI if reflect == -1 else 0} ${0 if reflect == -1 else PI}"/>
+      <origin xyz="0.0455 ${reflect * -0.018} 0" rpy="0 ${PI if reflect == -1 else 0} ${0 if reflect == -1 else PI}"/>
       <geometry>
         <mesh filename="package://my_turtlebot_pkg/meshes/n20motor_centered.stl" scale="0.001 0.001 0.001"/>
@@ -162,4 +162,13 @@
       <material name="wheel_black"/>
     </visual>
+    <!-- Collision -->
+    <collision>
+      <origin xyz="0.0455 ${reflect * -0.018} 0"
+              rpy="0 ${PI if reflect == -1 else 0} ${0 if reflect == -1 else PI}"/>
+      <geometry>
+        <mesh filename="package://my_turtlebot_pkg/meshes/n20motor_centered.stl"
+            scale="0.001 0.001 0.001"/>
+      </geometry>
+    </collision>
     <inertial>
       <mass value="${motor_mass}"/>
@@ -315,4 +324,5 @@
     <pose>0 0 0 0 0 0</pose>
     <topic>scan</topic>
+    <gz_frame_id>lidar_link</gz_frame_id>
     <update_rate>10</update_rate>
     <lidar>
